File: PCBs/Motor_Shield_v1/Motor_Shield_v1.kicad_pcb (KiCad board)
At the start: 4 copper layers, 68.6 x 53.3 mm, 32 parts, among them J1 Power, J2 Digital/PWM, J3 Analog, J4 Digital/PWM

Commit message: revise PCB to handle Motor Current
Routing:
- net +24V: track 84.4 -> 15.8 mm
- net Net-(11-OUT_2): track 73.9 -> 80.5 mm
- net Net-(1-OUT_2): track 59.9 -> 63.3 mm
- net Net-(11-OUT_1): track 60.0 -> 58.6 mm
- net Net-(1-OUT_1): track 65.1 -> 64.2 mm
- added copper zone on B.Cu, net +24V
Other:
- board text removed: "JLCJLCJLCJLC"
